File: x180.kicad_sch (KiCad schematic)
At the start: 73 parts, among them J1 U180 Header, J2 Conn_01x06_Pin, U1 ATF1502AS-7A, U2 ADG734, U3 ADG734, U4 ADG734, U5 ADG734

Commit message: REV B: redesign with resistor networks
Parts:
- removed R1: 4k3, Resistor_SMD:R_0805_2012Metric, symbol Device:R
- removed R10, R28, R3, R31, R4, R5, R6, R7: 20k, Resistor_SMD:R_0805_2012Metric, symbol Device:R
- removed R11, R12, R26, R27, R29, R30, R8, R9: 160k, Resistor_SMD:R_0805_2012Metric, symbol Device:R
- removed R17, R18, R25: 10k, Resistor_SMD:R_0805_2012Metric, symbol Device:R
- removed R19, R22, R23: 37k5, Resistor_SMD:R_0805_2012Metric, symbol Device:R
- removed R2: 6k2, Resistor_SMD:R_0805_2012Metric, symbol Device:R
- removed R20, R21: 16k7, Resistor_SMD:R_0805_2012Metric, symbol Device:R
- removed R24: 24k, Resistor_SMD:R_0805_2012Metric, symbol Device:R
- added +12, +5, -12: TestPoint_Small, MiDi:TestPoint_Pad_D1.0mm, symbol Connector:TestPoint
- added C14: 100n, Capacitor_SMD:C_1206_3216Metric, symbol Device:C_Small
- added JP1: SolderJumper_3_Open, Jumper:SolderJumper-3_P1.3mm_Open_RoundedPad1.0x1.5mm, symbol Jumper:SolderJumper_3_Open
- added R.A1, R.A2, R.B1, R.B2, R.J1, R.J2: 300k, Resistor_SMD:R_0805_2012Metric, symbol Device:R
- added R.I1, R.I2: 100k, Resistor_SMD:R_0805_2012Metric, symbol Device:R
- added RN1, RN2, RN3, RN4, RN5, RN6, RN7, RN8: OSOP 20k, MiDi:SSOP-20_3.9x8.7mm_P0.635mm, symbol MiDi:RN_OSOP_10
- added RN10: LT5400 10k, Package_SO:MSOP-8-1EP_3x3mm_P0.65mm_EP1.68x1.88mm, symbol Device:R_Pack04
- added RN11, RN9: OSOP 5k, MiDi:SSOP-20_3.9x8.7mm_P0.635mm, symbol Device:R_Pack10
- R13, R14, R15, R16, R32, R33, R34, R35, R36, R37, R38, R39, R40: value 100R -> 22R
Connections:
- net PIN58 AGND2 is gone; now on net AGND: J1.58 (AGND2), U3.14 (S3B), U3.17 (S4B), U3.4 (S1B), U3.7 (S2B)
- net PIN59 AGND3 is gone; now on net GND: J1.59 (AGND3), U4.14 (S3B), U4.4 (S1B), U4.7 (S2B), U5.4 (S1B), U5.7 (S2B)
- net +12_REF: now also +12.1, RN1.3 (R3.1), RN1.5 (R5.1), RN10.1 (R1.1), RN10.2 (R2.1), RN3.3 (R3.1), RN5.6 (R6.1), RN5.8 (R8.1), RN7.8 (R8.1), RN9.2 (R2.1), RN9.4 (R4.1)
- net -12_REF: now also -12.1, RN1.6 (R6.1), RN1.8 (R8.1), RN10.3 (R3.1), RN10.4 (R4.1), RN11.1 (R1.1), RN3.8 (R8.1), RN5.3 (R3.1), RN5.5 (R5.1), RN7.3 (R3.1)
- net GND: now also J1.1 (GND), J1.17 (GND), J1.60 (GND), J1.61 (GND), J1.62 (GND), JP1.3 (B), RN10.9 (R1.2)
- net GND2: now also JP1.1 (A); no longer C1.1, C10.1, C3.1, C6.1, U2.5 (VSS), U3.5 (VSS), U4.5 (VSS), U5.5 (VSS)
- net PIN11 50K OUT: now also RN7.17 (R4.2), RN8.14 (R7.2), RN8.17 (R4.2); no longer J1.12 (50K_MID1)
- net PIN15 +5_SUM: now also C14.1, RN11.10 (R10.1), RN11.9 (R9.1)
- net PIN16 +5_REF: now also +5.1, C14.2, RN11.19 (R2.2)
- net PIN18 LADEXT: now also R.B1.1, RN1.2 (R2.1), RN3.2 (R2.1)
- net PIN19 LADT2: now also R.I2.1, RN5.9 (R9.1), RN7.9 (R9.1)
- net PIN2 +12_SUM: now also RN9.10 (R10.1), RN9.6 (R6.1), RN9.8 (R8.1), RN9.9 (R9.1)
- net PIN21 LADT1: now also R.I1.2, RN2.12 (R9.2), RN4.12 (R9.2)
- net PIN23 LAD: now also R.J2.2, RN6.11 (R10.2), RN8.11 (R10.2)
- net PIN3 +12_GND: now also RN9.18 (R3.2), RN9.20 (R1.2)
- net PIN6 50K IN: now also RN1.4 (R4.1), RN1.7 (R7.1), RN2.7 (R7.1)
- net PIN9 -12_SUM: now also RN10.5 (R4.2), RN10.6 (R3.2), RN10.7 (R2.2), RN10.8 (R1.2)
- net +12ref2 20k: now reaches U3.13 (D3)
- net +12ref2 20k: now also RN6.13 (R8.2), RN8.13 (R8.2)
- net +12ref1 80k: now reaches U2.3 (D1)
- net +12ref1 80k: now also RN4.16 (R5.2)
- net -12ref1 80k: now reaches U2.13 (D3)
- net -12ref1 80k: now also RN4.15 (R6.2)
- net -12ref2 80k: now reaches U3.8 (D2)
- net -12ref2 80k: now also RN8.16 (R5.2)
- net +12ref1 20k: now reaches U2.8 (D2)
- net +12ref1 20k: now also RN2.18 (R3.2), RN4.18 (R3.2)
- net +12ref2 80k: now reaches U3.18 (D4)
- net +12ref2 80k: now also RN8.15 (R6.2)
- net -12ref1 20k: now reaches U2.18 (D4)
- net -12ref1 20k: now also RN2.13 (R8.2), RN4.13 (R8.2)
- net -12ref2 20k: now reaches U3.3 (D1)
- net -12ref2 20k: now also RN6.18 (R3.2), RN8.18 (R3.2)
- net PIN57 AGND1 renamed AGND
- new net: RN2.20 (R1.2), RN4.20 (R1.2), RN5.1 (R1.1), RN7.1 (R1.1)
- new net: RN5.20 (R1.2), RN6.1 (R1.1), RN7.20 (R1.2), RN8.1 (R1.1)
- new net: RN3.15 (R6.2), RN4.6 (R6.1)
- new net: RN11.11 (R10.2), RN11.13 (R8.2)
- new net: RN11.12 (R9.2), RN11.14 (R7.2), RN11.17 (R4.2)
- new net: RN11.15 (R6.2), RN11.16 (R5.2)
- new net: RN11.18 (R3.2), RN11.20 (R1.2)
- new net: RN11.2 (R2.1), RN11.4 (R4.1), RN11.7 (R7.1)
- new net: RN11.3 (R3.1), RN11.5 (R5.1)
- new net: RN11.6 (R6.1), RN11.8 (R8.1)
- new net: R.A1.1, R.I1.1, R.J1.1, RN1.1 (R1.1), RN1.10 (R10.1), RN1.9 (R9.1), RN3.1 (R1.1), RN3.10 (R10.1), RN3.9 (R9.1)
- new net: R.A1.2, R.A2.1
- new net: RN5.13 (R8.2), RN6.8 (R8.1), RN7.13 (R8.2), RN8.8 (R8.1)
- new net: RN5.15 (R6.2), RN6.6 (R6.1)
- new net: RN2.16 (R5.2), RN3.5 (R5.1)
- new net: RN1.16 (R5.2), RN2.5 (R5.1)
- new net: RN1.13 (R8.2), RN2.8 (R8.1), RN3.13 (R8.2), RN4.8 (R8.1)
- new net: RN3.16 (R5.2), RN4.5 (R5.1)
- new net: RN1.18 (R3.2), RN2.3 (R3.1), RN3.18 (R3.2), RN4.3 (R3.1)
- new net: RN5.18 (R3.2), RN6.3 (R3.1), RN7.18 (R3.2), RN8.3 (R3.1)
- new net: RN2.11 (R10.2), RN4.11 (R10.2), RN5.10 (R10.1), RN7.10 (R10.1)
- new net: RN5.11 (R10.2), RN6.10 (R10.1), RN7.11 (R10.2), RN8.10 (R10.1)
- new net: RN1.15 (R6.2), RN2.6 (R6.1)
- new net: R.A2.2, R.B2.2, R.I2.2, RN6.12 (R9.2), RN6.19 (R2.2), RN6.20 (R1.2), RN8.12 (R9.2), RN8.19 (R2.2), RN8.20 (R1.2)
- new net: RN7.16 (R5.2), RN8.5 (R5.1)
- new net: RN6.16 (R5.2), RN7.5 (R5.1)
- new net: RN9.1 (R1.1), RN9.3 (R3.1), RN9.5 (R5.1), RN9.7 (R7.1)
- new net: RN9.11 (R10.2), RN9.13 (R8.2), RN9.14 (R7.2), RN9.16 (R5.2)
- new net: RN9.12 (R9.2), RN9.15 (R6.2), RN9.17 (R4.2), RN9.19 (R2.2)
- new net: RN2.15 (R6.2), RN3.6 (R6.1)
- new net: RN5.16 (R5.2), RN6.5 (R5.1)
- new net: RN6.17 (R4.2), RN7.4 (R4.1), RN8.4 (R4.1)
- new net: RN5.19 (R2.2), RN6.2 (R2.1), RN7.19 (R2.2), RN8.2 (R2.1)
- new net: RN2.19 (R2.2), RN4.19 (R2.2), RN5.2 (R2.1), RN7.2 (R2.1)
- new net: R.J1.2, R.J2.1
- new net: RN1.19 (R2.2), RN2.2 (R2.1), RN3.19 (R2.2), RN4.2 (R2.1)
- new net: RN1.20 (R1.2), RN2.1 (R1.1), RN3.20 (R1.2), RN4.1 (R1.1)
- new net: RN1.12 (R9.2), RN2.9 (R9.1), RN3.12 (R9.2), RN4.9 (R9.1)
- new net: RN1.14 (R7.2), RN2.14 (R7.2), RN3.7 (R7.1)
- new net: RN3.17 (R4.2), RN4.14 (R7.2), RN4.17 (R4.2), RN5.4 (R4.1), RN5.7 (R7.1), RN6.7 (R7.1)
- new net: RN2.17 (R4.2), RN3.4 (R4.1), RN4.4 (R4.1)
- new net: RN7.14 (R7.2), RN8.7 (R7.1)
- new net: RN5.14 (R7.2), RN6.14 (R7.2), RN7.7 (R7.1)
- new net: RN1.11 (R10.2), RN2.10 (R10.1), RN3.11 (R10.2), RN4.10 (R10.1)
- new net: RN1.17 (R4.2), RN2.4 (R4.1)
- new net: R.B1.2, R.B2.1
- new net: RN7.15 (R6.2), RN8.6 (R6.1)
- new net: RN6.15 (R6.2), RN7.6 (R6.1)
- new net: RN5.12 (R9.2), RN6.9 (R9.1), RN7.12 (R9.2), RN8.9 (R9.1)
- new net: RN5.17 (R4.2), RN6.4 (R4.1)
- new net: RN3.14 (R7.2), RN4.7 (R7.1)
- new net VSS: C1.1, C10.1, C3.1, C6.1, JP1.2 (C), U2.5 (VSS), U3.5 (VSS), U4.5 (VSS), U5.5 (VSS)
- no-connect marks 5 -> 0
Other:
- note added: "16k667"
- note added: "20k"
- note added: "30k:12k5"
- note added: "37k5"
- note added: "37k5 S4 37k5 S16 +12ref1 20k -12ref2 20k Input 50k +12ref1 80k -12ref2 80k -12ref1 80k +12ref2 80k Input 50k -12ref1 20k +12ref2 20k 16k7 S64 16k7 S16 37k5 S64"
- note added: "50k"
- note added: "5k:5k"
- note added: "5k:7k5"
- note added: "80k"
- note added: "A B C D E F G H I J"
- note added: "Alternative: 2k with 12 resistors"
- note added: "C0G"
- note added: "RN1"
- note added: "RN1..8 OSOP 10x20k"
- note added: "RN1..8 usage"
- note added: "RN2"
- note added: "RN3"
- note added: "RN4"
- note added: "RN5"
- note added: "RN6"
- note added: "RN7"
- note added: "RN8"
- moved on the sheet: C1, C10, C11, C12, C13, C2, C3, C4, C5, C6, C7, C8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

Commit message: REV C: optimized for low stray capacitance & back to discrete resistors
Parts:
- removed R.A1, R.A2, R.B1, R.B2, R.J1, R.J2: 300k, Resistor_SMD:R_0805_2012Metric, symbol Device:R
- removed R.I1, R.I2: 100k, Resistor_SMD:R_0805_2012Metric, symbol Device:R
- removed RN1, RN2, RN3, RN4, RN5, RN6, RN7, RN8: OSOP 20k, MiDi:SSOP-20_3.9x8.7mm_P0.635mm, symbol MiDi:RN_OSOP_10
- added JP1: SolderJumper_3_Open, MiDi:SolderJumper-3_P0.7mm_Open_RoundedPad0.7x0.4mm, symbol Jumper:SolderJumper_3_Open
- added R10, R11, R12, R13, R14, R15, R20, R21, R22, R23, R28, R29, R30, R31, R32, R33, R6, R7, R8, R9: 20k, Resistor_SMD:R_1206_3216Metric, symbol Device:R
- added R34, R36, R39, R42, R43: 10k, Resistor_SMD:R_1206_3216Metric, symbol Device:R
- added R35, R38, R41: 37k5, Resistor_SMD:R_0805_2012Metric, symbol Device:R
- added R37, R40: 16k7, Resistor_SMD:R_0805_2012Metric, symbol Device:R
- C1: renamed from C2; now not fitted
- C2: renamed from C4; now not fitted
- C3: renamed from C7; now not fitted
- C4: renamed from C12; now not fitted
- C5: renamed from C1; now not fitted
- C6: renamed from C3; now not fitted
- C7: renamed from C6; now not fitted
- C8: renamed from C10; now not fitted
- JP2: renamed from JP1; footprint Jumper:SolderJumper-3_P1.3mm_Open_RoundedPad1.0x1.5mm -> MiDi:SolderJumper-3_P0.7mm_Open_RoundedPad0.7x0.4mm
- renumbered +5 to +1, +12 to +2, -12 to -1, C9 to C10, C13 to C12, C14 to C13, C5 to C14, C8 to C9, R13 to R1, R15 to R16, R34 to R17, R37 to R18, R39 to R19, R32 to R2, R16 to R24, R35 to R25, R38 to R26, R40 to R27, R14 to R3, R33 to R4, R36 to R5, RN9 to RN1, RN11 to RN2, RN10 to RN3, S6 to S1, S11 to S10, S4 to S11, S1 to S12, S17 to S13, S9 to S2, S7 to S3, S8 to S4, S0 to S5, S10 to S6, S5 to S7, S2 to S8, S3 to S9, U2 to U1, U3 to U2, U4 to U3, U5 to U4, U1 to U5
Connections:
- net +12_REF: now also R20.2, R28.2, R29.2, R33.2
- net +12ref1 20k: now also R28.1
- net +12ref1 80k: now also R23.1
- net +12ref2 20k: now also R33.1
- net +12ref2 80k: now also R32.1
- net -12_REF: now also R10.2, R11.2, R15.2, R6.2
- net -12ref1 20k: now also R10.1
- net -12ref1 80k: now also R9.1
- net -12ref2 20k: now also R15.1
- net -12ref2 80k: now also R14.1
- net GND: no longer RN3.9 (R1.2)
- net PIN11 50K OUT: now also R43.1
- net PIN18 LADEXT: now also R35.1
- net PIN19 LADT2: now also R37.1
- net PIN21 LADT1: now also R40.1
- net PIN23 LAD: now also R41.2
- net PIN3 +12_GND: now also RN3.9 (R1.2)
- net PIN6 50K IN: now also R34.2
- net VCC: now also JP1.3 (B); no longer C1.2, C2.2, C3.2, C4.2, U1.16 (VDD), U2.16 (VDD), U3.16 (VDD), U4.16 (VDD)
- new net: R31.1, R32.2
- new net: R30.1, R31.2
- new net: R42.1, R43.2
- new net: R21.1, R22.2
- new net: R20.1, R21.2
- new net: R36.1, R39.2
- new net: R34.1, R36.2
- new net: R39.1, R42.2
- new net: R29.1, R30.2
- new net: R13.1, R14.2
- new net: R12.1, R13.2
- new net: R35.2, R37.2, R38.1
- new net: R22.1, R23.2
- new net: R8.1, R9.2
- new net: R38.2, R40.2, R41.1
- new net: R11.1, R12.2
- new net: R6.1, R7.2
- new net: R7.1, R8.2
- new net VDD: C1.2, C2.2, C3.2, C4.2, JP1.2 (C), U1.16 (VDD), U2.16 (VDD), U3.16 (VDD), U4.16 (VDD)
- new net VDD2: J1.52 (VDD2), JP1.1 (A)
Other:
- note added: "37k5: 2x75k piggybacked 16k7: 2x33k2 or 3x49k9 piggybacked"
- note added: "Alternative: 2x20k piggybacked"
- note removed: "16k667"
- note removed: "20k"
- note removed: "37k5"
- note removed: "37k5 S4 37k5 S16 +12ref1 20k -12ref2 20k Input 50k +12ref1 80k -12ref2 80k -12ref1 80k +12ref2 80k Input 50k -12ref1 20k +12ref2 20k 16k7 S64 16k7 S16 37k5 S64"
- note removed: "50k"
- note removed: "80k"
- note removed: "A B C D E F G H I J"
- note removed: "RN1"
- note removed: "RN1..8 OSOP 10x20k"
- note removed: "RN1..8 usage"
- note removed: "RN2"
- note removed: "RN3"
- note removed: "RN4"
- note removed: "RN5"
- note removed: "RN6"
- note removed: "RN7"
- note removed: "RN8"
- moved on the sheet: C13, C14, JP2
